Commit message: Add MuJoCo simulation with closed kinematic chains
- generate_mjcf.py builds the MJCF from geometry.yaml and dynamics.yaml:
  ball-jointed distal links tied to the platforms with connect equalities,
  central spherical joint, 9 position servos named like the ros2_control
  joints, finger collision hulls; masses estimated from the meshes (PLA)
- ros2_control tag selects mujoco_ros2_control/MujocoSystemInterface when
  ninedof.launch.py is started with sim:=mujoco
- forward kinematics wraps the angles to (-pi, pi]
- docs/nota_diseno_torsion.md: near-free torsion of platform 2 found with
  the CAD geometry and a parametric study of leg arrangements

Co-Authored-By: Claude Opus 5.5 <noreply@anthropic.com>
Claude-Session: https://claude.ai/code/session_011xKvdqfJ6fTy5kGUX9oYMQ

File: src/ninedof_description/urdf/ninedof.ros2_control.xacro (robot description, xacro)
@@ -2,8 +2,14 @@
 <!-- ros2_control interfaces of the 9 linear actuators (position commanded). -->
 <robot xmlns:xacro="http://www.ros.org/wiki/xacro">
-  <xacro:macro name="ninedof_ros2_control" params="legs stroke hardware_plugin">
+  <xacro:macro name="ninedof_ros2_control" params="legs stroke hardware_plugin headless:=false">
     <ros2_control name="NineDofSystem" type="system">
       <hardware>
         <plugin>${hardware_plugin}</plugin>
+        <xacro:if value="${hardware_plugin == 'mujoco_ros2_control/MujocoSystemInterface'}">
+          <!-- MJCF generated by scripts/generate_mjcf.py: closed chains, 9 position servos -->
+          <param name="mujoco_model">$(find ninedof_description)/mujoco/scene.xml</param>
+          <param name="headless">${headless}</param>
+          <param name="sim_speed_factor">1.0</param>
+        </xacro:if>
       </hardware>
       <xacro:ninedof_actuators legs="${legs}" stroke="${stroke}"/>

File: src/ninedof_description/urdf/ninedof.urdf.xacro (robot description, xacro)
@@ -15,4 +15,6 @@
        ideal actuators (the commanded position becomes the measured one). -->
   <xacro:arg name="hardware_plugin" default="mock_components/GenericSystem"/>
+  <!-- Only used with mujoco_ros2_control/MujocoSystemInterface -->
+  <xacro:arg name="headless" default="false"/>
   <xacro:property name="geometry_file" value="$(find ninedof_description)/config/geometry.yaml"/>
   <xacro:property name="g" value="${xacro.load_yaml(geometry_file)['ninedof']}"/>
@@ -113,4 +115,5 @@
   <xacro:include filename="$(find ninedof_description)/urdf/ninedof.ros2_control.xacro"/>
   <xacro:ninedof_ros2_control legs="${g['legs']}" stroke="${stroke}"
-                              hardware_plugin="$(arg hardware_plugin)"/>
+                              hardware_plugin="$(arg hardware_plugin)"
+                              headless="$(arg headless)"/>
 </robot>

Commit message: Pick-and-place demo with reorientation in MuJoCo
- ninedof_mujoco: SimStatePublisher plugin for mujoco_ros2_control (qpos and
  object pose topics, virtual grasp on /mujoco/grasp), pick_place_demo node
  (workspace check of every pose and interpolated path, grasp switching,
  qpos recording, final verification), render_video (1080p 30 fps mp4 via
  MUJOCO_GL=osmesa, geometry overlay) and pick_place.launch.py
- pick-and-place scene: robot hanging upside down, 12x12x24 mm block,
  30 deg turn (-10 -> +20 deg), heights inside the stroke window
- offline twin of the controller and the grasp for tests
- ninedof.launch.py: mujoco_scene and mujoco_plugins arguments
- Dockerfile: libosmesa6, ffmpeg and the MuJoCo Python bindings
- docs: video, key frames and design findings

Result in simulation: block placed 1.9 mm / 3.7 deg from the target.

Co-Authored-By: Claude Opus 5.5 <noreply@anthropic.com>
Claude-Session: https://claude.ai/code/session_011xKvdqfJ6fTy5kGUX9oYMQ

File: src/ninedof_description/urdf/ninedof.ros2_control.xacro (robot description, xacro)
@@ -2,5 +2,5 @@
 <!-- ros2_control interfaces of the 9 linear actuators (position commanded). -->
 <robot xmlns:xacro="http://www.ros.org/wiki/xacro">
-  <xacro:macro name="ninedof_ros2_control" params="legs stroke hardware_plugin headless:=false">
+  <xacro:macro name="ninedof_ros2_control" params="legs stroke hardware_plugin headless:=false mujoco_scene:=scene.xml">
     <ros2_control name="NineDofSystem" type="system">
       <hardware>
@@ -8,5 +8,5 @@
         <xacro:if value="${hardware_plugin == 'mujoco_ros2_control/MujocoSystemInterface'}">
           <!-- MJCF generated by scripts/generate_mjcf.py: closed chains, 9 position servos -->
-          <param name="mujoco_model">$(find ninedof_description)/mujoco/scene.xml</param>
+          <param name="mujoco_model">$(find ninedof_description)/mujoco/${mujoco_scene}</param>
           <param name="headless">${headless}</param>
           <param name="sim_speed_factor">1.0</param>

File: src/ninedof_description/urdf/ninedof.urdf.xacro (robot description, xacro)
@@ -17,4 +17,5 @@
   <!-- Only used with mujoco_ros2_control/MujocoSystemInterface -->
   <xacro:arg name="headless" default="false"/>
+  <xacro:arg name="mujoco_scene" default="scene.xml"/>  <!-- file in ninedof_description/mujoco -->
   <xacro:property name="geometry_file" value="$(find ninedof_description)/config/geometry.yaml"/>
   <xacro:property name="g" value="${xacro.load_yaml(geometry_file)['ninedof']}"/>
@@ -116,4 +117,5 @@
   <xacro:ninedof_ros2_control legs="${g['legs']}" stroke="${stroke}"
                               hardware_plugin="$(arg hardware_plugin)"
-                              headless="$(arg headless)"/>
+                              headless="$(arg headless)"
+                              mujoco_scene="$(arg mujoco_scene)"/>
 </robot>
